Commit message: success!

File: go2_navigation_sim/FAST_LIO_ROS2/config/robot.urdf.xacro (robot description, xacro)
@@ -7,5 +7,5 @@
     <parent link="base_link" />
     <child link="lidar_link" />
-    <origin xyz="0 0 0.0" rpy="0 0 0" />
+    <origin xyz="0 0 0.5" rpy="0 0 0" />
   </joint>
   <!--
@@ -21,5 +21,5 @@
     <parent link="lidar_link" />
     <child link="livox_frame" />
-    <origin xyz="0 0 0.5" rpy="0 0 0" />
+    <origin xyz="0 0 0.0" rpy="0 0 0" />
   </joint>
   <link name="gnss_link"> </link>
